Commit message: movimiento

File: hexapod_javi_sim/urdf/javi.urdf.xacro (robot description, xacro)
@@ -67,5 +67,5 @@
     <!-- Leg macro -->
     <xacro:macro name="leg" params="side position x y angle axis">
-        <!-- leg position -->
+        <!-- leg position
         <joint name="leg_center_joint_${side}${position}" type="fixed">
             <origin xyz="${x} ${y} 0.0" rpy="0.0 0.0 0.0"/>
@@ -83,8 +83,9 @@
             </inertial>
         </link>
+        -->
         <!-- coxa -->
         <joint name="coxa_joint_${side}${position}" type="revolute">
-            <origin xyz="0.0 0.0 0.0" rpy="0.0 0.0 ${angle}"/>
-            <parent link="leg_center_${side}${position}"/>
+            <origin xyz="${x} ${y} 0.0" rpy="0.0 0.0 ${angle}"/>
+            <parent link="body_link"/>
             <child link="coxa_${side}${position}"/>
             <axis xyz="0.0 0.0 1.0"/>
