Commit message: renamed all files

File: h_robix_description/urdf/javi.urdf.xacro (robot description, xacro)
@@ -33,5 +33,5 @@
             <origin xyz="-0.034138 0.204808 -0.031029" rpy="${pi/2} 0.0 0.0"/>
             <geometry>
-                <mesh filename="package://hexapod_javi_sim/meshes/base_link.stl" scale="0.001 0.001 0.001"/>
+                <mesh filename="package://h_robix_description/meshes/base_link.stl" scale="0.001 0.001 0.001"/>
             </geometry>
             <material name="">
@@ -42,5 +42,5 @@
             <origin xyz="0.0 0.0 0.0" rpy="0.0 0.0 0.0"/>
             <geometry>
-                <mesh filename="package://hexapod_javi_sim/meshes/base_link.stl" scale="0.001 0.001 0.001"/>
+                <mesh filename="package://h_robix_description/meshes/base_link.stl" scale="0.001 0.001 0.001"/>
             </geometry>
             <material name="">
@@ -105,5 +105,5 @@
                 <origin xyz="0.012 0.0 0.0" rpy="0.0 0.0 ${pi/2}"/>
                 <geometry>
-                    <mesh filename="package://hexapod_javi_sim/meshes/coxa_link.stl" scale="0.001 0.001 0.001"/>
+                    <mesh filename="package://h_robix_description/meshes/coxa_link.stl" scale="0.001 0.001 0.001"/>
                 </geometry>
                 <material name="">
@@ -114,5 +114,5 @@
                 <origin xyz="0.012 0.0 0.0" rpy="0.0 0.0 ${pi/2}" />
                 <geometry>
-                    <mesh filename="package://hexapod_javi_sim/meshes/coxa_link.stl" scale="0.001 0.001 0.001"/>
+                    <mesh filename="package://h_robix_description/meshes/coxa_link.stl" scale="0.001 0.001 0.001"/>
                 </geometry>
                 <material name="">
@@ -154,5 +154,5 @@
                 <origin xyz="0.066 -0.09827 -0.024054" rpy="0.0 0.0 ${-pi/2}"/>
                 <geometry>
-                    <mesh filename="package://hexapod_javi_sim/meshes/femur_link.stl" scale="0.001 0.001 0.001"/>
+                    <mesh filename="package://h_robix_description/meshes/femur_link.stl" scale="0.001 0.001 0.001"/>
                 </geometry>
                 <material name="">
@@ -163,5 +163,5 @@
                 <origin xyz="0.066 -0.09827 -0.024054" rpy="0.0 0.0 ${-pi/2} " />
                 <geometry>
-                    <mesh filename="package://hexapod_javi_sim/meshes/femur_link.stl" scale="0.001 0.001 0.001"/>
+                    <mesh filename="package://h_robix_description/meshes/femur_link.stl" scale="0.001 0.001 0.001"/>
                 </geometry>
                 <material name="">
@@ -200,5 +200,5 @@
                 <origin xyz="0.0185 0.030551 -0.002466" rpy="${-pi*3/4} ${pi/2} 0.0"/>
                 <geometry>
-                    <mesh filename="package://hexapod_javi_sim/meshes/tibia_link.stl" scale="0.001 0.001 0.001"/>
+                    <mesh filename="package://h_robix_description/meshes/tibia_link.stl" scale="0.001 0.001 0.001"/>
                 </geometry>
                 <material name="">
@@ -209,5 +209,5 @@
                 <origin xyz="0.0185 0.030551 -0.002466" rpy="${-pi*3/4} ${pi/2} 0.0" />
                 <geometry>
-                    <mesh filename="package://hexapod_javi_sim/meshes/tibia_link.stl" scale="0.001 0.001 0.001"/>
+                    <mesh filename="package://h_robix_description/meshes/tibia_link.stl" scale="0.001 0.001 0.001"/>
                 </geometry>
                 <material name="">
